File: PCB/POWER.kicad_sch (KiCad schematic)
At the start: 32 parts, among them IC100 AP63203WU-7, J100 2604-3102, Q100 CSD19537Q3, Q101 BSS138, U100 TPS26631RGE

Commit message: Cambio del footprint Efuse
- Se ha cambiado el footorint de chip Efuse debido a que el utilizado no habia stock en JLCPCB
- Se ha creado los archivos de configuracion para JLCPCB
Parts:
- removed U100: TPS26631RGE, Package_DFN_QFN:Texas_RGE0024H_VQFN-24-1EP_4x4mm_P0.5mm_EP2.7x2.7mm_ThermalVias, symbol Power_Management:TPS26631RGE
- added U100: TPS26631PWP, Package_SO:HTSSOP-20-1EP_4.4x6.5mm_P0.65mm_EP3.4x6.5mm_Mask2.96x2.96mm_ThermalVias, symbol Power_Management:TPS26631PWP
Connections:
- net +24V: now also U100.16 (PGTH), U100.18 (OUT), U100.19 (OUT), U100.20 (OUT)
- net FLT: now also U100.15 (~{FLT})
- net GND: now also U100.12 (MODE), U100.21 (GND), U100.9 (GND)
- net INPUT: now also U100.6 (IN_SYS)
- net at R103.1: now also U100.11 (ILIM)
- net at R100.2, R101.1: now also U100.7 (UVLO)
- net at R101.2, R102.1: now also U100.8 (OVP)
- net at Q100.3 (D): now also U100.1 (IN), U100.2 (IN), U100.3 (IN)
- net at Q100.2 (G), Q101.3 (D): now also U100.4 (B_GATE)
- net at Q101.1 (G): now also U100.5 (DRV)
- net at C101.2: now also U100.10 (dVdT)
Changed lines of the file:
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@@
 	)
 	(symbol
-		(lib_id "Power_Management:TPS26631RGE")
+		(lib_id "Power_Management:TPS26631PWP")
 		(at 108.458 82.042 0)
 		(unit 1)
@@
 		(fields_autoplaced yes)
 		(property "Reference" "U100"
-			(at 110.6521 61.976 0)
+			(at 110.6521 61.468 0)
 			(effects
 				(font
@@
 			)
 		)
-		(property "Value" "TPS26631RGE"
-			(at 110.6521 64.516 0)
+		(property "Value" "TPS26631PWP"
+			(at 110.6521 64.008 0)
 			(effects
 				(font
@@
 			)
 		)
-		(property "Footprint" "Package_DFN_QFN:Texas_RGE0024H_VQFN-24-1EP_4x4mm_P0.5mm_EP2.7x2.7mm_ThermalVias"
+		(property "Footprint" "Package_SO:HTSSOP-20-1EP_4.4x6.5mm_P0.65mm_EP3.4x6.5mm_Mask2.96x2.96mm_ThermalVias"
 			(at 108.458 113.792 0)
 			(effects
@@
 			)
 		)
-		(property "Description" "60V, 6A Power Limiting, Surge Protection Industrial eFuse, Adjustable Overvoltage cut-off, Active Current Limiting with Pulse current support, VQFN-24"
+		(property "Description" "60V, 6A Power Limiting, Surge Protection Industrial eFuse, Adjustable Overvoltage cut-off, Active Current Limiting with Pulse current support, HTTSOP-20"
 			(at 108.458 82.042 0)
 			(effects
@@
 			)
 		)
-		(property "LCSC" "C1850273"
+		(property "LCSC" "C2832195"
 			(at 108.458 82.042 0)
 			(effects
@@
 			)
 		)
+		(pin "13"
+		)
+		(pin "18"
+		)
+		(pin "15"
+		)
+		(pin "5"
+		)
 		(pin "11"
-		)
-		(pin "6"
 		)
 		(pin "10"
 		)
-		(pin "21"
-		)
-		(pin "23"
-		)
-		(pin "12"
-		)
-		(pin "9"
-		)
-		(pin "24"
+		(pin "20"
 		)
 		(pin "17"
 		)
+		(pin "21"
+		)
 		(pin "2"
-		)
-		(pin "13"
-		)
-		(pin "4"
-		)
-		(pin "7"
 		)
 		(pin "8"
@@
 		(pin "1"
 		)
-		(pin "19"
-		)
-		(pin "22"
-		)
 		(pin "14"
 		)
-		(pin "18"
+		(pin "9"
 		)
-		(pin "25"
+		(pin "16"
 		)
-		(pin "5"
-		)
-		(pin "15"
+		(pin "19"
 		)
 		(pin "3"
 		)
-		(pin "16"
+		(pin "12"
 		)
-		(pin "20"
+		(pin "7"
+		)
+		(pin "4"
+		)
+		(pin "6"
 		)
 		(instances
-			(project "PCB-Cuarto"
+			(project ""
 				(path "/118ffa26-3c65-424a-af71-04338c4de0b0/e2751aaa-40ab-491e-8724-b4cb7cd2712b"
 					(reference "U100")
